File: pcb/out/rx2/rx2.kicad_pcb (KiCad board)
At the start: 2 copper layers, 86.8 x 73.8 mm, 31 parts, among them J1 PWR+VREF, J2 ADC OUT, K1 TCT40-16R, K2 TCT40-16R, U1 MCP6004

Commit message: เตรียมเก็บชุดข้อมูลรอบสอง: อาเรย์สี่เหลี่ยม + เก็บท่าทางอย่างเป็นระบบ
ย้าย RX ไปมุมทั้งสี่ของ plate_mini แล้ว (TL=GPIO35 TR=GPIO34 BL=GPIO32
BR=GPIO33 TX=GPIO18 ตรงกลาง) เดิม RX เรียงเป็นเส้นนอนบนบอร์ดทดลอง
ซึ่งแยกบน-ล่างไม่ได้เลยในทางฟิสิกส์ ตอนนี้ได้ทิศแนวตั้งมาด้วย

rig2.py เก็บรูปทรงอาเรย์ไว้ที่เดียว เบสไลน์ 110 มม. ทั้งสองแกน
ที่ 40 kHz คลื่นยาว 8.6 มม. แยกแยะได้ 4.5 องศาทั้งสองแกน
ผลต่างเวลาสูงสุดระหว่างคู่ทแยง 454 ไมโครวินาที

pose_cue.py วาดหุ่นไม้ขีดบอกท่าพร้อมนับถอยหลัง 8 ท่า วน 4 รอบ ท่าละ 6 วินาที
ไม่ยุ่งกับการอัด รันคู่ขนานได้ กล้อง depth เป็นคนบอกเฉลยอยู่แล้ว
ตัวนี้แค่ทำให้คนหน้ากล้องเปลี่ยนท่าอย่างเป็นระบบ

เหตุผลที่ต้องมี: วัดแล้วพบว่าโมเดลรอบแรกอยู่ใต้เพดาน 'รู้แค่ตำแหน่ง'
ทั้งสองแกน สาเหตุไม่ใช่โมเดลแต่เป็นข้อมูล เพราะท่าทางแทบไม่เคยเปลี่ยน
ขณะที่ตำแหน่งคงที่ พอตำแหน่งอธิบายภาพได้เกือบหมด โมเดลก็ไม่มีเหตุผล
ต้องเรียนอย่างอื่น รอบนี้จึงแยกท่ากับตำแหน่งออกจากกันในข้อมูล

บันทึกไว้ตรง ๆ ว่าตาราง 80x60 ไม่ได้เพิ่มความละเอียดจริง หนึ่งช่องกว้าง
0.73 องศา แต่ความเบลอทางฟิสิกส์กินราว 6 ช่อง ที่ทำได้คือท่าทาง ซึ่งเป็น
การเปลี่ยนแปลงระดับ 40-60 องศา ใหญ่กว่าขีดจำกัดสิบเท่า
Routing:
- net 3V3: track 78.6 -> 337.8 mm
- net CH2_S2O: track 103.4 -> 36.4 mm
- net CH2_S2N: track 89.8 -> 45.4 mm
- net CH2_S1O: track 53.8 -> 72.4 mm
- net CH1_S1N: track 80.2 -> 65.0 mm
- net CH1_S1O: track 66.6 -> 56.2 mm
- net VREF: track 73.0 -> 81.2 mm
- net CH2_S1N: track 69.8 -> 73.4 mm
- net CH1_G: track 45.0 -> 48.6 mm
- net CH2_G1: track 3.00 -> 5.40 mm
- net CH1_G1: track 3.00 -> 5.40 mm
- net CH2_G2: track 3.20 -> 5.60 mm
- net CH1_S2N: track 54.6 -> 52.2 mm
- net CH1_G2: track 3.20 -> 5.60 mm
