File: pcb/out/main8/main8.kicad_sch (KiCad schematic)
At the start: 116 parts, among them K1 RX1, K2 RX2, K3 RX3, K4 RX4, K5 RX5, K6 RX6, K7 RX7, K8 RX8, T1 TX1, T2 TX2, T3 TX3, U1 1/2, U2 A, U3 A, U4 A, U5 A, U6 A

Commit message: pcb: แก้ผังที่นำเข้าแล้วแตกเป็นเส้น เพิ่มกรอบตัวถังบนบอร์ด และแพ็คเป็นซิป
**สาเหตุที่ผังเปิดใน EasyEDA แล้วเป็นเส้นลอย ๆ ไม่เป็นสัญลักษณ์**
ตัวต้านทานแนวนอน แนวตั้ง และแบบสลับขา ถูกยัดให้ใช้นิยามสัญลักษณ์ตัวเดียวกัน
ตัวที่บันทึกทีหลังทับตัวก่อนหน้า ขาของอีกสามทิศจึงไปโผล่ผิดที่ สายกับขา
ไม่บรรจบกัน โดนแบบนี้ 54 ตัวจาก 142 (คาปาและเทอร์มินอลก็เป็นแบบเดียวกัน)
แยกนิยามตามทิศของขา 1 แล้วใส่ตัวกันไว้ ถ้าชื่อเดียวกันถูกใช้กับสองรูปทรงจะหยุดทันที

**เพิ่มตัวตรวจพิกัด ซึ่งจับบั๊กข้างบนได้ตั้งแต่แรกถ้ามีมาก่อน**
ตัวตรวจเดิมดูว่า "ขาไหนควรอยู่เน็ตอะไร" ซึ่งผ่านหมดทั้ง 340 ขา
แต่ไม่ได้ดูว่า "สายไปบรรจบกับขาตรงพิกัดจริงหรือเปล่า"
ตัวใหม่จับได้ 50 ขาลอย ในนั้นมีรอยขาดจริงในผังด้วย ซึ่งภาพ SVG ก็ขาดตามไปด้วย
  ขาซ้ายของตัวป้อนกลับไม่ได้ต่อกับปมขาลบ (ทั้ง 16 สเตจ)
  คาปาปลายทางกับคาปากรองไฟไม่ได้ต่อกับปมที่ห้อยอยู่
เติมสายที่ขาดแล้ว ตอนนี้ทุกขาใน 340 จุดมีสายหรือป้ายมาบรรจบจริง
ขาที่ตั้งใจไม่ต่อ 23 ขา ใส่เครื่องหมายไม่ต่อให้ ไม่ให้โปรแกรมเตือนว่าลืม

**หน้ากระดาษ** เดิมเรียงทุกแผ่นลงล่างจนได้ 503 x 1956 มม. เปิดมาเป็นแถบผอม
เปลี่ยนเป็นวางเป็นคอลัมน์ และภาครับ 8 ช่องวางเป็นตาราง 2x4
ได้ 1386 x 766 มม. สัดส่วนใกล้เคียงกระดาษปกติ

**บอร์ดไม่มีเส้นกรอบตัวถังเลยแม้แต่เส้นเดียว** มีแต่แป้นกับตัวอักษร
geom.body() มีมานานแล้วแต่ตัวส่งออก KiCad ไม่เคยเรียกใช้
ประกอบไม่ได้เพราะมองไม่ออกว่าตัวไหนหันทางไหน และ 3D ก็โล่งเพราะไม่มีอะไรให้วาด
เพิ่มกรอบ 464 เส้น (116 ตัว x 4 ด้าน) และจุดบอกขา 1 ทุกตัว

**pack_kicad()** แพ็ค .kicad_pro + .kicad_sch + .kicad_pcb เป็นซิปเดียว
ชื่อไฟล์ทั้งสามต้องตรงกัน ตัวนำเข้าจึงจะผูกผังกับบอร์ดเข้าด้วยกันได้
Parts:
- removed C1G1, C1G2, C2G1, C2G2, C3G1, C3G2, C4G1, C4G2, C5G1, C5G2, C6G1, C6G2, C7G1, C7G2, C8G1, C8G2, CD1, CD2, CD3, CD4, CD5, CD6, CV1: 100nF, symbol ultrasonic:C
- removed C1I, C2I, C3I, C4I, C5I, C6I, C7I, C8I: 10nF, symbol ultrasonic:C
- removed C1O, C2O, C3O, C4O, C5O, C6O, C7O, C8O: 1nF, symbol ultrasonic:C
- removed CB1, CB2: 10uF, symbol ultrasonic:C
- removed CF: 100uF, symbol ultrasonic:C
- removed JP: 5V เข้า, symbol ultrasonic:TERM2
- removed K1: RX1, symbol ultrasonic:TERM2
- removed K2: RX2, symbol ultrasonic:TERM2
- removed K3: RX3, symbol ultrasonic:TERM2
- removed K4: RX4, symbol ultrasonic:TERM2
- removed K5: RX5, symbol ultrasonic:TERM2
- removed K6: RX6, symbol ultrasonic:TERM2
- removed K7: RX7, symbol ultrasonic:TERM2
- removed K8: RX8, symbol ultrasonic:TERM2
- removed R1B, R2B, R3B, R4B, R5B, R6B, R7B, R8B: 1M, symbol ultrasonic:R
- removed R1F1, R1F2, R2F1, R2F2, R3F1, R3F2, R4F1, R4F2, R5F1, R5F2, R6F1, R6F2, R7F1, R7F2, R8F1, R8F2: 33k, symbol ultrasonic:R
- removed R1G1, R1G2, R1O, R2G1, R2G2, R2O, R3G1, R3G2, R3O, R4G1, R4G2, R4O, R5G1, R5G2, R5O, R6G1, R6G2, R6O, R7G1, R7G2, R7O, R8G1, R8G2, R8O: 1k, symbol ultrasonic:R
- removed RF: 10R, symbol ultrasonic:R
- removed RT1, RT2, RT3: 100R, symbol ultrasonic:R
- removed RV1, RV2: 10k, symbol ultrasonic:R
- removed T1: TX1, symbol ultrasonic:TERM2
- removed T2: TX2, symbol ultrasonic:TERM2
- removed T3: TX3, symbol ultrasonic:TERM2
- added C1G1, C1G2, C2G1, C2G2, C3G1, C3G2, C4G1, C4G2, C5G1, C5G2, C6G1, C6G2, C7G1, C7G2, C8G1, C8G2, CD1, CD2, CD3, CD4, CD5, CD6, CV1: 100nF, symbol ultrasonic:C_U
- added C1I, C2I, C3I, C4I, C5I, C6I, C7I, C8I: 10nF, symbol ultrasonic:C_L
- added C1O, C2O, C3O, C4O, C5O, C6O, C7O, C8O: 1nF, symbol ultrasonic:C_U
- added CB1, CB2: 10uF, symbol ultrasonic:C_U
- added CF: 100uF, symbol ultrasonic:C_U
- added JP: 5V เข้า, symbol ultrasonic:TERM2_R
- added K1: RX1, symbol ultrasonic:TERM2_R
- added K2: RX2, symbol ultrasonic:TERM2_R
- added K3: RX3, symbol ultrasonic:TERM2_R
- added K4: RX4, symbol ultrasonic:TERM2_R
- added K5: RX5, symbol ultrasonic:TERM2_R
- added K6: RX6, symbol ultrasonic:TERM2_R
- added K7: RX7, symbol ultrasonic:TERM2_R
- added K8: RX8, symbol ultrasonic:TERM2_R
- added R1B, R2B, R3B, R4B, R5B, R6B, R7B, R8B: 1M, symbol ultrasonic:R_D
- added R1F1, R1F2, R2F1, R2F2, R3F1, R3F2, R4F1, R4F2, R5F1, R5F2, R6F1, R6F2, R7F1, R7F2, R8F1, R8F2: 33k, symbol ultrasonic:R_R
- added R1G1, R1G2, R2G1, R2G2, R3G1, R3G2, R4G1, R4G2, R5G1, R5G2, R6G1, R6G2, R7G1, R7G2, R8G1, R8G2: 1k, symbol ultrasonic:R_U
- added R1O, R2O, R3O, R4O, R5O, R6O, R7O, R8O: 1k, symbol ultrasonic:R_L
- added RF: 10R, symbol ultrasonic:R_L
- added RT1, RT2, RT3: 100R, symbol ultrasonic:R_L
- added RV1, RV2: 10k, symbol ultrasonic:R_U
- added T1: TX1, symbol ultrasonic:TERM2_L
- added T2: TX2, symbol ultrasonic:TERM2_L
- added T3: TX3, symbol ultrasonic:TERM2_L
Connections:
- no-connect marks 0 -> 23

Commit message: pcb: แก้ชื่อนิยามสัญลักษณ์ ที่ทำให้ผังเข้ามาแต่สาย ไม่มีชิ้นส่วนเลย
นำเข้าแล้วเห็นแต่เส้นเขียวลอย ๆ ไม่มีตัวต้านทาน ไม่มีชิป ไม่มีอะไรสักตัว

สาเหตุ: นิยามสัญลักษณ์ตั้งชื่อว่า "C_L" แต่ชิ้นส่วนอ้างถึง "ultrasonic:C_L"
รูปแบบ KiCad กำหนดให้ชื่อในนิยามต้องมีชื่อคลังนำหน้าด้วย ให้ตรงกับที่อ้างถึง
ส่วนชื่อของ unit ข้างในใช้ชื่อเปล่า ผมใส่คลังนำหน้าแค่ฝั่งที่อ้างถึงฝั่งเดียว
ตัวนำเข้าหานิยามไม่เจอ เลยทิ้งสัญลักษณ์ทั้ง 142 ตัว เหลือแต่สาย 371 เส้น

เพิ่ม check_names() ซึ่งเป็นตัวตรวจที่จะจับบั๊กนี้ได้ตั้งแต่แรก
ตัวตรวจเดิมสองตัวผ่านหมด เพราะตัวหนึ่งดูว่าขาอยู่เน็ตถูกไหม อีกตัวดูว่า
สายบรรจบกับขาตรงพิกัดไหม ทั้งคู่ไม่ได้ดูว่าปลายทางจะหานิยามเจอไหม
รวมเป็นสามชั้น: เน็ตถูก · พิกัดบรรจบ · หานิยามเจอ

แก้ตัวอักษรนำหน้าเลขอ้างอิงในนิยามด้วย เดิมตัดชื่อ 4 ตัวแรกไปเทียบ
ซึ่งไม่ตรงกับชื่อที่มีคำต่อท้ายบอกทิศ ทุกตัวเลยได้ U หมด
Connections:
- net A3V3: now also CD2.1, CD3.1, CD4.1, CD5.1, CD6.1, CF.1, RF.2, RV1.1, U2.4, U3.4, U4.4, U5.4, U6.4
- net GND: now also C1G1.2, C1G2.2, C1O.2, C2G1.2, C2G2.2, C2O.2, C3G1.2, C3G2.2, C3O.2, C4G1.2, C4G2.2, C4O.2, C5G1.2, C5G2.2, C5O.2, C6G1.2, C6G2.2, C6O.2, C7G1.2, C7G2.2, C7O.2, C8G1.2, C8G2.2, C8O.2, CB1.2, CB2.2, CD1.2, CD2.2, CD3.2, CD4.2, CD5.2, CD6.2, CF.2, CV1.2, JA.1, JB.19, JP.2, RV2.2, T1.2, T2.2, T3.2, U1.7, U2.11, U3.11, U4.11, U5.11, U6.11
- net MCU3V3: now also JA.3, JB.20, RF.1
- net MID: now also RV1.2, RV2.1, U6.3
- net P5V: now also CB1.1, CD1.1, JB.18, JP.1, U1.14
- net RX1_ADC: now also C1O.1, JA.16, R1O.2
- net RX2_ADC: now also C2O.1, JA.15, R2O.2
- net RX3_ADC: now also C3O.1, JA.14, R3O.2
- net RX4_ADC: now also C4O.1, JA.13, R4O.2
- net RX5_ADC: now also C5O.1, R5O.2
- net RX6_ADC: now also C6O.1, JA.11, R6O.2
- net RX7_ADC: now also C7O.1, JA.10, R7O.2
- net RX8_ADC: now also C8O.1, JA.9, R8O.2
- net TX1_IN: now also JB.14, U1.1
- net TX2_IN: now also JB.15, U1.13
- net TX3_IN: now also JB.16, U1.5
- net VREF: now also CB2.1, CV1.1, R1B.2, R2B.2, R3B.2, R4B.2, R5B.2, R6B.2, R7B.2, R8B.2, U6.1, U6.10, U6.12, U6.13, U6.14, U6.2, U6.5, U6.6, U6.7, U6.8, U6.9
- new net: R7F1.2, R7G1.1, U5.2
- new net: C7G1.1, R7G1.2
- new net: C4I.2, R4B.1, U3.10
- new net: R4F1.1, U3.12, U3.8
- new net: R4F1.2, R4G1.1, U3.9
- new net: R5F2.1, R5O.1, U4.7
- new net: R2F1.1, U2.12, U2.8
- new net: R2F1.2, R2G1.1, U2.9
- new net: C1I.2, R1B.1, U2.3
- new net: C6I.2, R6B.1, U4.10
- new net: R6F1.1, U4.12, U4.8
- new net: R6F1.2, R6G1.1, U4.9
- new net: C3I.2, R3B.1, U3.3
- new net: C8I.2, R8B.1, U5.10
- new net: R8F1.1, U5.12, U5.8
- new net: R8F1.2, R8G1.1, U5.9
- new net: R2F2.1, R2O.1, U2.14
- new net: R3F1.1, U3.1, U3.5
- new net: R3F2.2, R3G2.1, U3.6
- new net: R3F2.1, R3O.1, U3.7
- new net: C5I.1, K5.1
- new net: R5F2.2, R5G2.1, U4.6
- new net: C5G2.1, R5G2.2
- new net: C2I.2, R2B.1, U2.10
- new net: R2F2.2, R2G2.1, U2.13
- new net: R5F1.1, U4.1, U4.5
- new net: RT3.2, T3.1
- new net: C8G2.1, R8G2.2
- new net: R1F2.1, R1O.1, U2.7
- new net: R1F2.2, R1G2.1, U2.6
- new net: R6F2.2, R6G2.1, U4.13
- new net: C6G2.1, R6G2.2
- new net: R7F2.2, R7G2.1, U5.6
- new net: C7G2.1, R7G2.2
- new net: R8F2.2, R8G2.1, U5.13
- new net: C1I.1, K1.1
- new net: C3I.1, K3.1
- new net: R4F2.1, R4O.1, U3.14
- new net: C3G2.1, R3G2.2
- new net: U1.2, U1.3
- new net: RT1.1, U1.4
- new net: R5F1.2, R5G1.1, U4.2
- new net: C5G1.1, R5G1.2
- new net: C8G1.1, R8G1.2
- new net: C6G1.1, R6G1.2
- new net: R6F2.1, R6O.1, U4.14
- new net: R3F1.2, R3G1.1, U3.2
- new net: U1.11, U1.12
- new net: C7I.1, K7.1
- new net: R7F1.1, U5.1, U5.5
- new net: R7F2.1, R7O.1, U5.7
- new net: R8F2.1, R8O.1, U5.14
- new net: C2G1.1, R2G1.2
- new net: C4G1.1, R4G1.2
- new net: C4I.1, K4.1
- new net: R1F1.1, U2.1, U2.5
- new net: R1F1.2, R1G1.1, U2.2
- new net: C7I.2, R7B.1, U5.3
- new net: C1G1.1, R1G1.2
- new net: C1G2.1, R1G2.2
- new net: C2G2.1, R2G2.2
- new net: RT1.2, T1.1
- new net: C5I.2, R5B.1, U4.3
- new net: R4F2.2, R4G2.1, U3.13
- new net: C6I.1, K6.1
- new net: RT3.1, U1.8
- new net: RT2.2, T2.1
- new net: U1.6, U1.9
- new net: C2I.1, K2.1
- new net: C3G1.1, R3G1.2
- new net: RT2.1, U1.10
- new net: C4G2.1, R4G2.2
- new net: C8I.1, K8.1
